File: projects/Ramen80/Ramen80.kicad_pcb (KiCad board)
At the start: 2 copper layers, 364 x 140 mm, 306 parts, among them J1 USB4105-GF-A, J2 USB_C_RECEPTACLE, K1 KEYSW, K10 KEYSW, K11 KEYSW, K12 KEYSW, K13 KEYSW, K14 KEYSW, K15 KEYSW, K16 KEYSW, K17 KEYSW, K18 KEYSW, K19 KEYSW, K2 KEYSW, K20 KEYSW, K21 KEYSW, K22 KEYSW, K23 KEYSW, K24 KEYSW, K25 KEYSW, K26 KEYSW, K27 KEYSW, K28 KEYSW, K29 KEYSW, K3 KEYSW, K30 KEYSW, K31 KEYSW, K32 KEYSW, K33 KEYSW, K34 KEYSW, K35 KEYSW, K36 KEYSW, K37 KEYSW, K38 KEYSW, K39 KEYSW, K4 KEYSW, K40 KEYSW, K41 KEYSW, K42 KEYSW, K43 KEYSW, K44 KEYSW, K45 KEYSW, K46 KEYSW, K47 KEYSW, K48 KEYSW, K49 KEYSW, K5 KEYSW, K50 KEYSW, K51 KEYSW, K52 KEYSW, K53 KEYSW, K54 KEYSW, K55 KEYSW, K56 KEYSW, K57 KEYSW, K58 KEYSW, K59 KEYSW, K6 KEYSW, K60 KEYSW, K61 KEYSW, K62 KEYSW, K63 KEYSW, K64 KEYSW, K65 KEYSW, K66 KEYSW, K67 KEYSW, K68 KEYSW, K69 KEYSW, K7 KEYSW, K70 KEYSW, K71 KEYSW, K72 KEYSW, K73 KEYSW, K74 KEYSW, K75 KEYSW, K76 KEYSW, K77 KEYSW, K78 KEYSW, K79 KEYSW, K8 KEYSW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

Commit message: Fixes
Parts:
- moved R7 1.00 mm to (311.0, 144.0)
Routing:
- net /LED Matrix/SW1: track 855.9 -> 0.00 mm, vias 12 -> 0
- net /LED Matrix/2SW2: track 685.5 -> 0.00 mm, vias 15 -> 0
- net /LED Matrix/SW2: track 679.7 -> 0.00 mm, vias 15 -> 0
- net /LED Matrix/SW3: track 655.8 -> 0.00 mm, vias 16 -> 0
- net VCC: track 457.7 -> 0.00 mm, vias 4 -> 0
- net /PF7: track 432.5 -> 0.00 mm
- net /LED Matrix/2SW3: track 428.5 -> 0.00 mm, vias 19 -> 0
- net /LED Matrix/2SW8: track 415.0 -> 0.00 mm, vias 8 -> 0
- net /PF0: track 397.5 -> 0.00 mm, vias 2 -> 0
- net /LED Matrix/2SW1: track 391.8 -> 0.00 mm, vias 16 -> 0
- net /PF1: track 368.1 -> 0.00 mm, vias 2 -> 0
- net /PB1: track 342.7 -> 0.00 mm, vias 4 -> 0
- net /PE6: track 333.4 -> 0.00 mm, vias 2 -> 0
- net /PB0: track 322.2 -> 0.00 mm, vias 2 -> 0
- net /LED Matrix/2SW4: track 313.0 -> 0.00 mm, vias 8 -> 0
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
Commit message: Fixes
Parts:
- R4: moved to B.Cu
- R8: moved to F.Cu
- moved R11 244.9 mm to (385.0, 136.0), turned to -90 degrees
- moved R5 244.9 mm to (141.9, 165.2), turned to 180 degrees
- moved R12 187.3 mm to (314.0, 124.0)
- moved R6 187.3 mm to (131.9, 167.7)
- moved R4 79.1 mm to (313.4, 144.2), turned to 90 degrees
- moved R8 78.9 mm to (325.0, 66.0), turned to -90 degrees
- moved C16 44.3 mm to (373.4, 146.0), turned to 0 degrees
- moved C24 44.3 mm to (331.0, 133.0), turned to 90 degrees
- moved R7 0.47 mm to (311.4, 144.2)

Commit message: Fixes
Parts:
- R1, R2, R3: moved to B.Cu
- R10, R7, R9: moved to F.Cu
- moved R10 178.6 mm to (325.0, 62.0), turned to -90 degrees
- moved R2 170.4 mm to (188.1, 168.7), turned to 90 degrees
- moved R9 167.6 mm to (323.0, 62.0), turned to -90 degrees
- moved R1 166.0 mm to (197.9, 166.3), turned to 0 degrees
- moved R7 83.7 mm to (327.0, 62.0)
- moved R3 79.1 mm to (311.4, 144.2), turned to 90 degrees
- moved C24 9.67 mm to (326.2, 124.6)
- moved U3 7.11 mm to (194.3, 172.4)
- moved R8 5.66 mm to (321.0, 62.0)
- moved R12 4.41 mm to (312.2, 128.0)
- moved R5 1.60 mm to (140.7, 166.3)
- moved R6 1.36 mm to (131.0, 168.7)
- moved U2 1.36 mm to (137.2, 172.4)
- renumbered U3 to U2, U2 to U3
Routing:
- net /UCap: track 0.00 -> 9.35 mm
- net VCC: track 0.00 -> 6.53 mm
- net /USB C Receptacle/Cap+: track 0.00 -> 6.45 mm
- net Net-(J2-PadA5): track 0.00 -> 5.06 mm
- net Net-(J2-PadB5): track 0.00 -> 4.85 mm
- net /USB C Receptacle/Cap-: track 0.00 -> 2.69 mm
- net /PE2: track 0.00 -> 2.29 mm
- net GND: vias 1 -> 0

Commit message: Fixes
Parts:
- moved C11 16.9 mm to (369.5, 144.0)
- moved C16 14.0 mm to (373.0, 132.0)
- moved C13 13.7 mm to (373.0, 126.0)
- moved C10 12.8 mm to (369.5, 142.0)
- moved C18 12.5 mm to (373.0, 136.0), turned to 0 degrees
- moved C17 12.4 mm to (373.0, 134.0), turned to 0 degrees
- moved C2 11.6 mm to (369.5, 126.0)
- moved C9 9.51 mm to (369.5, 140.0), turned to 180 degrees
- moved C14 7.51 mm to (373.0, 128.0)
- moved C3 7.51 mm to (369.5, 128.0)
- moved C12 6.31 mm to (369.5, 146.0)
- moved C21 6.11 mm to (373.0, 142.0)
- moved C19 5.91 mm to (373.0, 138.0)
- moved C4 4.82 mm to (369.5, 130.0), turned to 180 degrees
- moved C5 4.76 mm to (369.5, 132.0), turned to 180 degrees
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Routing:
- net /USB C Receptacle/Cap-: track 2.69 -> 7.13 mm

Commit message: Fixed!
Connections:
- D1 pad 2: Net-(D16-Pad2) -> Net-(D1-Pad2)
- D10 pad 2: Net-(D7-Pad2) -> Net-(D10-Pad2)
- D11 pad 2: Net-(D6-Pad2) -> Net-(D11-Pad2)
- D12 pad 2: Net-(D5-Pad2) -> Net-(D12-Pad2)
- D13 pad 2: Net-(D4-Pad2) -> Net-(D13-Pad2)
- D14 pad 2: Net-(D3-Pad2) -> Net-(D14-Pad2)
- D15 pad 2: Net-(D2-Pad2) -> Net-(D15-Pad2)
- D16 pad 2: Net-(D1-Pad2) -> Net-(D16-Pad2)
- D17 pad 1: /PF5 -> /PF6
- D17 pad 2: Net-(D50-Pad2) -> Net-(D17-Pad2)
- D18 pad 1: /PF5 -> /PF6
- D18 pad 2: Net-(D48-Pad2) -> Net-(D18-Pad2)
- D19 pad 1: /PF5 -> /PF6
- D19 pad 2: Net-(D46-Pad2) -> Net-(D19-Pad2)
- D2 pad 2: Net-(D15-Pad2) -> Net-(D2-Pad2)
- D20 pad 1: /PF5 -> /PF6
- D20 pad 2: Net-(D44-Pad2) -> Net-(D20-Pad2)
- D21 pad 1: /PF5 -> /PF6
- D21 pad 2: Net-(D43-Pad2) -> Net-(D21-Pad2)
- D22 pad 1: /PF5 -> /PF6
- D22 pad 2: Net-(D40-Pad2) -> Net-(D22-Pad2)
- D23 pad 1: /PF5 -> /PF6
- D23 pad 2: Net-(D39-Pad2) -> Net-(D23-Pad2)
- D24 pad 1: /PF5 -> /PF6
- D24 pad 2: Net-(D35-Pad2) -> Net-(D24-Pad2)
- D25 pad 1: /PF5 -> /PF6
- D25 pad 2: Net-(D36-Pad2) -> Net-(D25-Pad2)
- D26 pad 2: Net-(D32-Pad2) -> Net-(D26-Pad2)
- D27 pad 2: Net-(D31-Pad2) -> Net-(D27-Pad2)
- D28 pad 2: Net-(D26-Pad2) -> Net-(D28-Pad2)
- D29 pad 2: Net-(D28-Pad2) -> Net-(D29-Pad2)
- D3 pad 2: Net-(D13-Pad2) -> Net-(D3-Pad2)
- D30 pad 2: Net-(D24-Pad2) -> Net-(D30-Pad2)
- D31 pad 2: Net-(D21-Pad2) -> Net-(D31-Pad2)
- D32 pad 2: Net-(D19-Pad2) -> Net-(D32-Pad2)
- D33 pad 2: Net-(D18-Pad2) -> Net-(D33-Pad2)
- D34 pad 2: Net-(D49-Pad2) -> Net-(D34-Pad2)
- D35 pad 2: Net-(D47-Pad2) -> Net-(D35-Pad2)
- D36 pad 2: Net-(D45-Pad2) -> Net-(D36-Pad2)
- D37 pad 2: Net-(D42-Pad2) -> Net-(D37-Pad2)
- D38 pad 2: Net-(D41-Pad2) -> Net-(D38-Pad2)
- D39 pad 2: Net-(D37-Pad2) -> Net-(D39-Pad2)
- D4 pad 2: Net-(D14-Pad2) -> Net-(D4-Pad2)
- D40 pad 2: Net-(D38-Pad2) -> Net-(D40-Pad2)
- D41 pad 2: Net-(D34-Pad2) -> Net-(D41-Pad2)
- D42 pad 1: /PF6 -> /PF5
- D42 pad 2: Net-(D33-Pad2) -> Net-(D42-Pad2)
- D43 pad 1: /PF6 -> /PF5
- D43 pad 2: Net-(D29-Pad2) -> Net-(D43-Pad2)
- D44 pad 1: /PF6 -> /PF5
- D44 pad 2: Net-(D30-Pad2) -> Net-(D44-Pad2)
- D45 pad 1: /PF6 -> /PF5
- D45 pad 2: Net-(D27-Pad2) -> Net-(D45-Pad2)
- D46 pad 1: /PF6 -> /PF5
- D46 pad 2: Net-(D25-Pad2) -> Net-(D46-Pad2)
- D47 pad 1: /PF6 -> /PF5
- D47 pad 2: Net-(D23-Pad2) -> Net-(D47-Pad2)
- D48 pad 1: /PF6 -> /PF5
- D48 pad 2: Net-(D22-Pad2) -> Net-(D48-Pad2)
- D49 pad 1: /PF6 -> /PF5
- D49 pad 2: Net-(D20-Pad2) -> Net-(D49-Pad2)
- D5 pad 2: Net-(D12-Pad2) -> Net-(D5-Pad2)
- D50 pad 1: /PF6 -> /PF5
- D50 pad 2: Net-(D17-Pad2) -> Net-(D50-Pad2)
- D51 pad 2: Net-(D63-Pad2) -> Net-(D51-Pad2)
- D52 pad 2: Net-(D61-Pad2) -> Net-(D52-Pad2)
- D53 pad 2: Net-(D62-Pad2) -> Net-(D53-Pad2)
- D54 pad 2: Net-(D60-Pad2) -> Net-(D54-Pad2)
- D55 pad 2: Net-(D59-Pad2) -> Net-(D55-Pad2)
- D56 pad 2: Net-(D58-Pad2) -> Net-(D56-Pad2)
- D58 pad 2: Net-(D56-Pad2) -> Net-(D58-Pad2)
- D59 pad 2: Net-(D55-Pad2) -> Net-(D59-Pad2)
- D6 pad 2: Net-(D11-Pad2) -> Net-(D6-Pad2)
- D60 pad 2: Net-(D54-Pad2) -> Net-(D60-Pad2)
- D61 pad 2: Net-(D53-Pad2) -> Net-(D61-Pad2)
- D62 pad 2: Net-(D52-Pad2) -> Net-(D62-Pad2)
- D63 pad 2: Net-(D51-Pad2) -> Net-(D63-Pad2)
- D64 pad 2: Net-(D76-Pad2) -> Net-(D64-Pad2)
- D65 pad 2: Net-(D75-Pad2) -> Net-(D65-Pad2)
- D66 pad 2: Net-(D74-Pad2) -> Net-(D66-Pad2)
- D67 pad 2: Net-(D73-Pad2) -> Net-(D67-Pad2)
- D68 pad 2: Net-(D72-Pad2) -> Net-(D68-Pad2)
- D69 pad 2: Net-(D71-Pad2) -> Net-(D69-Pad2)
- D7 pad 2: Net-(D10-Pad2) -> Net-(D7-Pad2)
- D71 pad 2: Net-(D69-Pad2) -> Net-(D71-Pad2)
- D72 pad 2: Net-(D68-Pad2) -> Net-(D72-Pad2)
- D73 pad 2: Net-(D67-Pad2) -> Net-(D73-Pad2)
- D74 pad 2: Net-(D66-Pad2) -> Net-(D74-Pad2)
- D75 pad 2: Net-(D65-Pad2) -> Net-(D75-Pad2)
- D76 pad 2: Net-(D64-Pad2) -> Net-(D76-Pad2)
- D77 pad 2: Net-(D87-Pad2) -> Net-(D77-Pad2)
- D78 pad 2: Net-(D86-Pad2) -> Net-(D78-Pad2)
- D79 pad 2: Net-(D85-Pad2) -> Net-(D79-Pad2)
- D8 pad 2: Net-(D9-Pad2) -> Net-(D8-Pad2)
- D80 pad 2: Net-(D84-Pad2) -> Net-(D80-Pad2)
- D81 pad 2: Net-(D83-Pad2) -> Net-(D81-Pad2)
- D83 pad 2: Net-(D81-Pad2) -> Net-(D83-Pad2)
- D84 pad 2: Net-(D80-Pad2) -> Net-(D84-Pad2)
- D85 pad 2: Net-(D79-Pad2) -> Net-(D85-Pad2)
- D86 pad 2: Net-(D78-Pad2) -> Net-(D86-Pad2)
- D87 pad 2: Net-(D77-Pad2) -> Net-(D87-Pad2)
- D9 pad 2: Net-(D8-Pad2) -> Net-(D9-Pad2)
- LED1 pad 4: /LED Matrix/CS16 -> /LED Matrix/CS1
- LED10 pad 4: /LED Matrix/CS7 -> /LED Matrix/CS10
- LED11 pad 4: /LED Matrix/CS6 -> /LED Matrix/CS11
- LED12 pad 4: /LED Matrix/CS5 -> /LED Matrix/CS12
- LED13 pad 4: /LED Matrix/CS4 -> /LED Matrix/CS13
- LED14 pad 4: /LED Matrix/CS3 -> /LED Matrix/CS14
- LED15 pad 4: /LED Matrix/CS2 -> /LED Matrix/CS15
- LED16 pad 4: /LED Matrix/CS1 -> /LED Matrix/CS16
- LED17 pad 1: /LED Matrix/2SW3 -> /LED Matrix/SW6
- LED17 pad 2: /LED Matrix/2SW1 -> /LED Matrix/SW4
- LED17 pad 3: /LED Matrix/2SW2 -> /LED Matrix/SW5
- LED17 pad 4: /LED Matrix/2CS5 -> /LED Matrix/CS1
- LED18 pad 1: /LED Matrix/2SW3 -> /LED Matrix/SW6
- LED18 pad 2: /LED Matrix/2SW1 -> /LED Matrix/SW4
- LED18 pad 3: /LED Matrix/2SW2 -> /LED Matrix/SW5
- LED18 pad 4: /LED Matrix/2CS6 -> /LED Matrix/CS2
- LED19 pad 1: /LED Matrix/2SW3 -> /LED Matrix/SW6
- LED19 pad 2: /LED Matrix/2SW1 -> /LED Matrix/SW4
- LED19 pad 3: /LED Matrix/2SW2 -> /LED Matrix/SW5
- LED19 pad 4: /LED Matrix/2CS2 -> /LED Matrix/CS3
- LED2 pad 4: /LED Matrix/CS15 -> /LED Matrix/CS2
- LED20 pad 1: /LED Matrix/SW9  -> /LED Matrix/SW6
- LED20 pad 2: /LED Matrix/SW7 -> /LED Matrix/SW4
- LED20 pad 3: /LED Matrix/SW8 -> /LED Matrix/SW5
- LED20 pad 4: /LED Matrix/CS14 -> /LED Matrix/CS4
- LED21 pad 1: /LED Matrix/SW9  -> /LED Matrix/SW6
- LED21 pad 2: /LED Matrix/SW7 -> /LED Matrix/SW4
- LED21 pad 3: /LED Matrix/SW8 -> /LED Matrix/SW5
- LED21 pad 4: /LED Matrix/CS9  -> /LED Matrix/CS5
- LED22 pad 1: /LED Matrix/SW9  -> /LED Matrix/SW6
- LED22 pad 2: /LED Matrix/SW7 -> /LED Matrix/SW4
- LED22 pad 3: /LED Matrix/SW8 -> /LED Matrix/SW5
- LED22 pad 4: /LED Matrix/CS8 -> /LED Matrix/CS6
- LED23 pad 1: /LED Matrix/SW9  -> /LED Matrix/SW6
- LED23 pad 2: /LED Matrix/SW7 -> /LED Matrix/SW4
- LED23 pad 3: /LED Matrix/SW8 -> /LED Matrix/SW5
- LED23 pad 4: /LED Matrix/CS6 -> /LED Matrix/CS7
- LED24 pad 1: /LED Matrix/SW9  -> /LED Matrix/SW6
- LED24 pad 2: /LED Matrix/SW7 -> /LED Matrix/SW4
- LED24 pad 3: /LED Matrix/SW8 -> /LED Matrix/SW5
- LED24 pad 4: /LED Matrix/CS3 -> /LED Matrix/CS8
- LED25 pad 1: /LED Matrix/SW9  -> /LED Matrix/SW6
- LED25 pad 2: /LED Matrix/SW7 -> /LED Matrix/SW4
- LED25 pad 3: /LED Matrix/SW8 -> /LED Matrix/SW5
- LED25 pad 4: /LED Matrix/CS2 -> /LED Matrix/CS9 
- LED26 pad 4: /LED Matrix/CS16 -> /LED Matrix/CS10
- LED27 pad 4: /LED Matrix/CS14 -> /LED Matrix/CS11
- LED29 pad 4: /LED Matrix/CS10 -> /LED Matrix/CS13
- LED3 pad 4: /LED Matrix/CS14 -> /LED Matrix/CS3
- LED30 pad 4: /LED Matrix/CS8 -> /LED Matrix/CS14
- LED31 pad 4: /LED Matrix/CS6 -> /LED Matrix/CS15
- LED32 pad 4: /LED Matrix/CS4 -> /LED Matrix/CS16
- LED33 pad 1: /LED Matrix/SW6 -> /LED Matrix/SW9 
- LED33 pad 2: /LED Matrix/SW4 -> /LED Matrix/SW7
- LED33 pad 3: /LED Matrix/SW5 -> /LED Matrix/SW8
- LED34 pad 1: /LED Matrix/2SW3 -> /LED Matrix/SW9 
- LED34 pad 2: /LED Matrix/2SW1 -> /LED Matrix/SW7
- LED34 pad 3: /LED Matrix/2SW2 -> /LED Matrix/SW8
- LED34 pad 4: /LED Matrix/2CS4 -> /LED Matrix/CS2
- LED35 pad 1: /LED Matrix/2SW3 -> /LED Matrix/SW9 
- LED35 pad 2: /LED Matrix/2SW1 -> /LED Matrix/SW7
- LED35 pad 3: /LED Matrix/2SW2 -> /LED Matrix/SW8
- LED35 pad 4: /LED Matrix/2CS3 -> /LED Matrix/CS3
- LED36 pad 1: /LED Matrix/2SW3 -> /LED Matrix/SW9 
- LED36 pad 2: /LED Matrix/2SW1 -> /LED Matrix/SW7
- LED36 pad 3: /LED Matrix/2SW2 -> /LED Matrix/SW8
- LED36 pad 4: /LED Matrix/2CS1 -> /LED Matrix/CS4
- LED37 pad 4: /LED Matrix/CS11 -> /LED Matrix/CS5
- LED38 pad 4: /LED Matrix/CS10 -> /LED Matrix/CS6
- LED4 pad 4: /LED Matrix/CS12 -> /LED Matrix/CS4
- LED40 pad 4: /LED Matrix/CS4 -> /LED Matrix/CS8
- LED41 pad 4: /LED Matrix/CS5 -> /LED Matrix/CS9 
- LED42 pad 4: /LED Matrix/CS1 -> /LED Matrix/CS10
- LED43 pad 1: /LED Matrix/SW6 -> /LED Matrix/SW9 
- LED43 pad 2: /LED Matrix/SW4 -> /LED Matrix/SW7
- LED43 pad 3: /LED Matrix/SW5 -> /LED Matrix/SW8
- LED43 pad 4: /LED Matrix/CS15 -> /LED Matrix/CS11
- LED44 pad 1: /LED Matrix/SW6 -> /LED Matrix/SW9 
- LED44 pad 2: /LED Matrix/SW4 -> /LED Matrix/SW7
- LED44 pad 3: /LED Matrix/SW5 -> /LED Matrix/SW8
- LED44 pad 4: /LED Matrix/CS13 -> /LED Matrix/CS14
- LED45 pad 1: /LED Matrix/SW6 -> /LED Matrix/2SW3
- LED45 pad 2: /LED Matrix/SW4 -> /LED Matrix/2SW1
- LED45 pad 3: /LED Matrix/SW5 -> /LED Matrix/2SW2
- LED45 pad 4: /LED Matrix/CS11 -> /LED Matrix/2CS1
- LED46 pad 1: /LED Matrix/SW6 -> /LED Matrix/2SW3
- LED46 pad 2: /LED Matrix/SW4 -> /LED Matrix/2SW1
- LED46 pad 3: /LED Matrix/SW5 -> /LED Matrix/2SW2
- LED46 pad 4: /LED Matrix/CS9  -> /LED Matrix/2CS2
- LED47 pad 1: /LED Matrix/SW6 -> /LED Matrix/2SW3
- LED47 pad 2: /LED Matrix/SW4 -> /LED Matrix/2SW1
- LED47 pad 3: /LED Matrix/SW5 -> /LED Matrix/2SW2
- LED47 pad 4: /LED Matrix/CS7 -> /LED Matrix/2CS3
- LED48 pad 1: /LED Matrix/SW6 -> /LED Matrix/2SW3
- LED48 pad 2: /LED Matrix/SW4 -> /LED Matrix/2SW1
- LED48 pad 3: /LED Matrix/SW5 -> /LED Matrix/2SW2
- LED48 pad 4: /LED Matrix/CS5 -> /LED Matrix/2CS4
- LED49 pad 1: /LED Matrix/SW6 -> /LED Matrix/2SW3
- LED49 pad 2: /LED Matrix/SW4 -> /LED Matrix/2SW1
- LED49 pad 3: /LED Matrix/SW5 -> /LED Matrix/2SW2
- LED49 pad 4: /LED Matrix/CS3 -> /LED Matrix/2CS5
- LED5 pad 4: /LED Matrix/CS13 -> /LED Matrix/CS5
- LED50 pad 1: /LED Matrix/SW6 -> /LED Matrix/2SW3
- LED50 pad 2: /LED Matrix/SW4 -> /LED Matrix/2SW1
- LED50 pad 3: /LED Matrix/SW5 -> /LED Matrix/2SW2
- LED50 pad 4: /LED Matrix/CS2 -> /LED Matrix/2CS6
- LED51 pad 1: /LED Matrix/2SW6 -> /LED Matrix/2SW3
- LED51 pad 2: /LED Matrix/2SW4 -> /LED Matrix/2SW1
- LED51 pad 3: /LED Matrix/2SW5 -> /LED Matrix/2SW2
- LED51 pad 4: /LED Matrix/2CS3 -> /LED Matrix/2CS7
- LED52 pad 1: /LED Matrix/2SW6 -> /LED Matrix/2SW3
- LED52 pad 2: /LED Matrix/2SW4 -> /LED Matrix/2SW1
- LED52 pad 3: /LED Matrix/2SW5 -> /LED Matrix/2SW2
- LED52 pad 4: /LED Matrix/2CS2 -> /LED Matrix/2CS8
- LED53 pad 4: /LED Matrix/2CS16 -> /LED Matrix/2CS9 
- LED54 pad 1: /LED Matrix/2SW6 -> /LED Matrix/2SW3
- LED54 pad 2: /LED Matrix/2SW4 -> /LED Matrix/2SW1
- LED54 pad 3: /LED Matrix/2SW5 -> /LED Matrix/2SW2
- LED54 pad 4: /LED Matrix/2CS1 -> /LED Matrix/2CS10
- LED55 pad 4: /LED Matrix/2CS15 -> /LED Matrix/2CS11
- LED56 pad 4: /LED Matrix/2CS14 -> /LED Matrix/2CS12
- LED58 pad 4: /LED Matrix/2CS12 -> /LED Matrix/2CS14
- LED59 pad 4: /LED Matrix/2CS11 -> /LED Matrix/2CS15
- LED6 pad 4: /LED Matrix/CS11 -> /LED Matrix/CS6
- LED60 pad 4: /LED Matrix/2CS10 -> /LED Matrix/2CS16
- LED61 pad 1: /LED Matrix/2SW3 -> /LED Matrix/2SW6
- LED61 pad 2: /LED Matrix/2SW1 -> /LED Matrix/2SW4
- LED61 pad 3: /LED Matrix/2SW2 -> /LED Matrix/2SW5
- LED61 pad 4: /LED Matrix/2CS9  -> /LED Matrix/2CS1
- LED62 pad 1: /LED Matrix/2SW3 -> /LED Matrix/2SW6
- LED62 pad 2: /LED Matrix/2SW1 -> /LED Matrix/2SW4
- LED62 pad 3: /LED Matrix/2SW2 -> /LED Matrix/2SW5
- LED62 pad 4: /LED Matrix/2CS8 -> /LED Matrix/2CS2
- LED63 pad 1: /LED Matrix/2SW3 -> /LED Matrix/2SW6
- LED63 pad 2: /LED Matrix/2SW1 -> /LED Matrix/2SW4
- LED63 pad 3: /LED Matrix/2SW2 -> /LED Matrix/2SW5
- LED63 pad 4: /LED Matrix/2CS7 -> /LED Matrix/2CS3
- LED64 pad 1: /LED Matrix/2SW9 -> /LED Matrix/2SW6
- LED64 pad 2: /LED Matrix/2SW7 -> /LED Matrix/2SW4
- LED64 pad 3: /LED Matrix/2SW8 -> /LED Matrix/2SW5
- LED64 pad 4: /LED Matrix/2CS1 -> /LED Matrix/2CS4
- LED65 pad 4: /LED Matrix/2CS15 -> /LED Matrix/2CS5
- LED66 pad 4: /LED Matrix/2CS14 -> /LED Matrix/2CS6
- LED67 pad 4: /LED Matrix/2CS13 -> /LED Matrix/2CS7
- LED68 pad 4: /LED Matrix/2CS11 -> /LED Matrix/2CS8
- LED69 pad 4: /LED Matrix/2CS12 -> /LED Matrix/2CS9 
- LED7 pad 4: /LED Matrix/CS10 -> /LED Matrix/CS7
- LED71 pad 4: /LED Matrix/2CS9  -> /LED Matrix/2CS11
- LED72 pad 4: /LED Matrix/2CS7 -> /LED Matrix/2CS12
- LED73 pad 4: /LED Matrix/2CS8 -> /LED Matrix/2CS13
- LED74 pad 4: /LED Matrix/2CS6 -> /LED Matrix/2CS14
- LED75 pad 4: /LED Matrix/2CS5 -> /LED Matrix/2CS15
- LED76 pad 1: /LED Matrix/2SW6 -> /LED Matrix/2SW9
- LED76 pad 2: /LED Matrix/2SW4 -> /LED Matrix/2SW7
- LED76 pad 3: /LED Matrix/2SW5 -> /LED Matrix/2SW8
- LED76 pad 4: /LED Matrix/2CS4 -> /LED Matrix/2CS1
- LED77 pad 4: /LED Matrix/2CS16 -> /LED Matrix/2CS2
- LED78 pad 4: /LED Matrix/2CS15 -> /LED Matrix/2CS3
- LED79 pad 4: /LED Matrix/2CS13 -> /LED Matrix/2CS4
- LED8 pad 4: /LED Matrix/CS9  -> /LED Matrix/CS8
- LED80 pad 4: /LED Matrix/2CS12 -> /LED Matrix/2CS7
- LED81 pad 4: /LED Matrix/2CS11 -> /LED Matrix/2CS9 
- LED83 pad 4: /LED Matrix/2CS9  -> /LED Matrix/2CS11
- LED84 pad 4: /LED Matrix/2CS7 -> /LED Matrix/2CS12
- LED85 pad 4: /LED Matrix/2CS4 -> /LED Matrix/2CS13
- LED86 pad 4: /LED Matrix/2CS3 -> /LED Matrix/2CS15
- LED87 pad 4: /LED Matrix/2CS2 -> /LED Matrix/2CS16
- LED9 pad 4: /LED Matrix/CS8 -> /LED Matrix/CS9 
- U2 pad 10: /LED Matrix/2SW8 -> /LED Matrix/SW8
- U2 pad 11: /LED Matrix/2SW9 -> /LED Matrix/SW9 
- U2 pad 16: /LED Matrix/2CS1 -> /LED Matrix/CS1
- U2 pad 17: /LED Matrix/2CS2 -> /LED Matrix/CS2
- U2 pad 18: /LED Matrix/2CS3 -> /LED Matrix/CS3
- U2 pad 19: /LED Matrix/2CS4 -> /LED Matrix/CS4
- U2 pad 2: /LED Matrix/2SW1 -> /LED Matrix/SW1
- U2 pad 21: /LED Matrix/2CS5 -> /LED Matrix/CS5
- U2 pad 22: /LED Matrix/2CS6 -> /LED Matrix/CS6
- U2 pad 23: /LED Matrix/2CS7 -> /LED Matrix/CS7
- U2 pad 24: /LED Matrix/2CS8 -> /LED Matrix/CS8
- U2 pad 25: /LED Matrix/2CS9  -> /LED Matrix/CS9 
- U2 pad 26: /LED Matrix/2CS10 -> /LED Matrix/CS10
- U2 pad 27: /LED Matrix/2CS11 -> /LED Matrix/CS11
- U2 pad 28: /LED Matrix/2CS12 -> /LED Matrix/CS12
- U2 pad 3: /LED Matrix/2SW2 -> /LED Matrix/SW2
- U2 pad 30: /LED Matrix/2CS13 -> /LED Matrix/CS13
- U2 pad 31: /LED Matrix/2CS14 -> /LED Matrix/CS14
- U2 pad 32: /LED Matrix/2CS15 -> /LED Matrix/CS15
- U2 pad 33: /LED Matrix/2CS16 -> /LED Matrix/CS16
- U2 pad 35: Net-(R6-Pad1) -> Net-(R2-Pad1)
- U2 pad 4: /LED Matrix/2SW3 -> /LED Matrix/SW3
- U2 pad 43: VCC -> GND
- U2 pad 47: Net-(R5-Pad2) -> Net-(R1-Pad2)
- U2 pad 6: /LED Matrix/2SW4 -> /LED Matrix/SW4
- U2 pad 7: /LED Matrix/2SW5 -> /LED Matrix/SW5
- U2 pad 8: /LED Matrix/2SW6 -> /LED Matrix/SW6
- U2 pad 9: /LED Matrix/2SW7 -> /LED Matrix/SW7
- U3 pad 10: /LED Matrix/SW8 -> /LED Matrix/2SW8
- U3 pad 11: /LED Matrix/SW9  -> /LED Matrix/2SW9
- U3 pad 16: /LED Matrix/CS1 -> /LED Matrix/2CS1
- U3 pad 17: /LED Matrix/CS2 -> /LED Matrix/2CS2
- U3 pad 18: /LED Matrix/CS3 -> /LED Matrix/2CS3
- U3 pad 19: /LED Matrix/CS4 -> /LED Matrix/2CS4
- U3 pad 2: /LED Matrix/SW1 -> /LED Matrix/2SW1
- U3 pad 21: /LED Matrix/CS5 -> /LED Matrix/2CS5
- U3 pad 22: /LED Matrix/CS6 -> /LED Matrix/2CS6
- U3 pad 23: /LED Matrix/CS7 -> /LED Matrix/2CS7
- U3 pad 24: /LED Matrix/CS8 -> /LED Matrix/2CS8
- U3 pad 25: /LED Matrix/CS9  -> /LED Matrix/2CS9 
- U3 pad 26: /LED Matrix/CS10 -> /LED Matrix/2CS10
- U3 pad 27: /LED Matrix/CS11 -> /LED Matrix/2CS11
- U3 pad 28: /LED Matrix/CS12 -> /LED Matrix/2CS12
- U3 pad 3: /LED Matrix/SW2 -> /LED Matrix/2SW2
- U3 pad 30: /LED Matrix/CS13 -> /LED Matrix/2CS13
- U3 pad 31: /LED Matrix/CS14 -> /LED Matrix/2CS14
- U3 pad 32: /LED Matrix/CS15 -> /LED Matrix/2CS15
- U3 pad 33: /LED Matrix/CS16 -> /LED Matrix/2CS16
- U3 pad 35: Net-(R2-Pad1) -> Net-(R6-Pad1)
- U3 pad 4: /LED Matrix/SW3 -> /LED Matrix/2SW3
- U3 pad 43: GND -> VCC
- U3 pad 47: Net-(R1-Pad2) -> Net-(R5-Pad2)
- U3 pad 6: /LED Matrix/SW4 -> /LED Matrix/2SW4
- U3 pad 7: /LED Matrix/SW5 -> /LED Matrix/2SW5
- U3 pad 8: /LED Matrix/SW6 -> /LED Matrix/2SW6
- U3 pad 9: /LED Matrix/SW7 -> /LED Matrix/2SW7
Routing:
- net GND: track 0.00 -> 80.3 mm, vias 0 -> 17
- net Net-(R2-Pad1): track 0.00 -> 2.28 mm
