File: projects/Ramen80/Ramen80.kicad_pcb (KiCad board)
At the start: 2 copper layers, 364 x 140 mm, 306 parts, among them J1 USB4105-GF-A, J2 USB_C_RECEPTACLE, K1 KEYSW, K10 KEYSW, K11 KEYSW, K12 KEYSW, K13 KEYSW, K14 KEYSW, K15 KEYSW, K16 KEYSW, K17 KEYSW, K18 KEYSW, K19 KEYSW, K2 KEYSW, K20 KEYSW, K21 KEYSW, K22 KEYSW, K23 KEYSW, K24 KEYSW, K25 KEYSW, K26 KEYSW, K27 KEYSW, K28 KEYSW, K29 KEYSW, K3 KEYSW, K30 KEYSW, K31 KEYSW, K32 KEYSW, K33 KEYSW, K34 KEYSW, K35 KEYSW, K36 KEYSW, K37 KEYSW, K38 KEYSW, K39 KEYSW, K4 KEYSW, K40 KEYSW, K41 KEYSW, K42 KEYSW, K43 KEYSW, K44 KEYSW, K45 KEYSW, K46 KEYSW, K47 KEYSW, K48 KEYSW, K49 KEYSW, K5 KEYSW, K50 KEYSW, K51 KEYSW, K52 KEYSW, K53 KEYSW, K54 KEYSW, K55 KEYSW, K56 KEYSW, K57 KEYSW, K58 KEYSW, K59 KEYSW, K6 KEYSW, K60 KEYSW, K61 KEYSW, K62 KEYSW, K63 KEYSW, K64 KEYSW, K65 KEYSW, K66 KEYSW, K67 KEYSW, K68 KEYSW, K69 KEYSW, K7 KEYSW, K70 KEYSW, K71 KEYSW, K72 KEYSW, K73 KEYSW, K74 KEYSW, K75 KEYSW, K76 KEYSW, K77 KEYSW, K78 KEYSW, K79 KEYSW, K8 KEYSW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

Commit message: Finished PCB
Parts:
- C1, C10, C11, C12, C13, C14, C15, C16, C17, C18, C19, C2, C20, C21, C22, C23, C24, C25, C26, C3, C4, C5, C6, C7, C8, C9: footprint Capacitor_SMD:C_0805_2012Metric -> RamenKeebs:C_0805
- D1, D10, D11, D12, D13, D14, D15, D16, D17, D18, D19, D2, D20, D21, D22, D23, D24, D25, D26, D27, D28, D29, D3, D30, D31, D32, D33, D34, D35, D36, D37, D38, D39, D4, D40, D41, D42, D43, D44, D45, D46, D47, D48, D49, D5, D50, D51, D52, D53, D54, D55, D56, D57, D58, D59, D6, D60, D61, D62, D63, D64, D65, D66, D67, D68, D69, D7, D70, D71, D72, D73, D74, D75, D76, D77, D78, D79, D8, D80, D81, D82, D83, D84, D85, D86, D87, D9: footprint keyboard_parts:D_SOD123_axial -> RamenKeebs:D_AXIAL
- J1: value USB4105-GF-A -> 6 Pin AVR
- J2: value USB_C_RECEPTACLE -> USB4505-03-0-A; footprint SamacSys_Parts:GCT_USB4105-GF-A -> RamenKeebs:USB4505-03-0-A
- K1, K10, K11, K12, K13, K14, K15, K16, K17, K18, K19, K2, K20, K21, K22, K23, K24, K25, K26, K27, K28, K29, K3, K30, K31, K32, K33, K34, K35, K36, K37, K38, K39, K4, K40, K41, K42, K43, K44, K45, K46, K47, K48, K49, K5, K50, K51, K52, K53, K54, K55, K56, K57, K58, K59, K6, K60, K61, K62, K63, K64, K65, K66, K67, K68, K69, K7, K70, K71, K72, K73, K74, K75, K76, K77, K78, K79, K8, K80, K81, K82, K83, K84, K85, K86, K87, K9: footprint keyswitches:Kailh_socket_MX_platemount -> RamenKeebs:KAILH_PLATEMOUNT
- R1, R10, R11, R12, R2, R3, R4, R5, R6, R7, R8, R9: footprint Resistor_SMD:R_0805_2012Metric -> RamenKeebs:R_0805
- U1: footprint Keebio-Parts:ATMEGA32U4-AU -> RamenKeebs:ATMEGA32U4-AUR
- moved J2 1.59 mm to (323.9, 50.4)
- moved R5 0.08 mm to (196.4, 165.3)
- moved R1 0.08 mm to (139.3, 165.3)
- turned K1 to 0 degrees
- turned K10 to 0 degrees
- turned K11 to 0 degrees
- turned K12 to 0 degrees
- turned K13 to 0 degrees
- turned K14 to 0 degrees
- turned K15 to 0 degrees
- turned K16 to 0 degrees
- turned K17 to 0 degrees
- turned K18 to 0 degrees
- turned K19 to 0 degrees
- turned K2 to 0 degrees
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Connections:
- J2 pad A1_B12: GND -> unconnected-(J2-PadA1_B12)
Routing:
- net /LED Matrix/2SW4: track 498.6 -> 856.1 mm, vias 21 -> 15
- net /PE6: track 386.0 -> 472.8 mm, vias 2 -> 8
- net /LED Matrix/SW9 : track 293.4 -> 378.4 mm, vias 11 -> 12
- net /LED Matrix/2CS14: track 329.2 -> 260.1 mm, vias 5 -> 4
- net /PD4: track 199.0 -> 267.5 mm, vias 2 -> 5
- net GND: track 95.9 -> 161.8 mm, vias 24 -> 37
- net /LED Matrix/SW4: track 528.2 -> 464.5 mm
- net /LED Matrix/2CS2: track 167.5 -> 229.8 mm, vias 5 -> 6
- net /LED Matrix/SW5: track 397.4 -> 459.2 mm, vias 26 -> 21
- net /LED Matrix/CS14: track 135.2 -> 195.5 mm
- net /PD2: track 319.1 -> 259.8 mm, vias 4 -> 3
- net /PB0: track 414.9 -> 357.0 mm, vias 2 -> 4
- net /LED Matrix/2CS3: track 246.1 -> 189.7 mm, vias 8 -> 4
- net /LED Matrix/2SW7: track 350.6 -> 400.3 mm, vias 12 -> 13
- net /PF1: track 400.2 -> 351.8 mm, vias 1 -> 3
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Other:
- board size 364 x 140 mm -> 355 x 133.2 mm

Commit message: Fixed all clearance violations
Routing:
- net GND: track 161.8 -> 227.7 mm, vias 37 -> 42
- net /PB2: track 412.2 -> 404.1 mm
- net /LED Matrix/2SW2: track 542.7 -> 539.7 mm
- net /LED Matrix/CS12: track 97.4 -> 99.3 mm
- net /LED Matrix/2SW8: track 365.4 -> 364.5 mm
- net /LED Matrix/SW5: track 459.2 -> 459.8 mm
- net /LED Matrix/CS11: track 161.8 -> 161.3 mm
