File: projects/Ramen80/Ramen80(Avr Prorgrammer).kicad_sch (KiCad schematic)
At the start: 1 part, among them J1 AVR_PROG

Commit message: Fixing the broke stuff
Parts:
- J1: value AVR_PROG -> USB4105-GF-A
Changed lines of the file:
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@@
   (symbol (lib_id "power:VCC") (at 68.58 35.56 90) (unit 1)
     (in_bom yes) (on_board yes) (fields_autoplaced)
-    (property "Reference" "#PWR036" (id 0) (at 72.39 35.56 0)
+    (property "Reference" "#PWR035" (id 0) (at 72.39 35.56 0)
       (effects (font (size 1.27 1.27)) hide)
     )
@@
   (symbol (lib_id "power:GND") (at 68.58 45.72 270) (unit 1)
     (in_bom yes) (on_board yes) (fields_autoplaced)
-    (property "Reference" "#PWR037" (id 0) (at 62.23 45.72 0)
+    (property "Reference" "#PWR036" (id 0) (at 62.23 45.72 0)
       (effects (font (size 1.27 1.27)) hide)
     )
@@
       (effects (font (size 1.27 1.27)) (justify left))
     )
-    (property "Value" "AVR_PROG" (id 1) (at 85.09 40.6399 0)
+    (property "Value" "USB4105-GF-A" (id 1) (at 85.09 40.6399 0)
       (effects (font (size 1.27 1.27)) (justify left))
     )

Commit message: Finished PCB
Parts:
- J1: value USB4105-GF-A -> 6 Pin AVR
Changed lines of the file:
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@@
   (title_block
     (title "Ramen80")
-    (date "2022-02-24")
+    (date "2022-03-05")
     (rev "v1.0.0")
     (company "Ramen Keebs")
@@
       (effects (font (size 1.27 1.27)) (justify left))
     )
-    (property "Value" "USB4105-GF-A" (id 1) (at 85.09 40.6399 0)
+    (property "Value" "6 Pin AVR" (id 1) (at 85.09 40.6399 0)
       (effects (font (size 1.27 1.27)) (justify left))
     )
