File: projects/Ramen80/Ramen80(Capacitor Grid).kicad_sch (KiCad schematic)
At the start: 6 parts

Commit message: Fixes continue...
Parts:
- C19, C21: value 0.1u -> 0.47f
- C20: value 0.1u -> 0.1f
- C23: value 4.7u -> 0.47f
- C24: value 1u -> 0.1f
Changed lines of the file:
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@@
       (effects (font (size 1.27 1.27)) (justify left))
     )
-    (property "Value" "0.1u" (id 1) (at 48.26 39.37 0)
+    (property "Value" "0.47f" (id 1) (at 48.26 39.37 0)
       (effects (font (size 1.27 1.27)) (justify left))
     )
@@
       (effects (font (size 1.27 1.27)) (justify left))
     )
-    (property "Value" "0.1u" (id 1) (at 57.15 39.37 0)
+    (property "Value" "0.1f" (id 1) (at 57.15 39.37 0)
       (effects (font (size 1.27 1.27)) (justify left))
     )
@@
       (effects (font (size 1.27 1.27)) (justify left))
     )
-    (property "Value" "0.1u" (id 1) (at 66.04 39.37 0)
+    (property "Value" "0.47f" (id 1) (at 66.04 39.37 0)
       (effects (font (size 1.27 1.27)) (justify left))
     )
@@
       (effects (font (size 1.27 1.27)) (justify left))
     )
-    (property "Value" "4.7u" (id 1) (at 83.82 39.37 0)
+    (property "Value" "0.47f" (id 1) (at 83.82 39.37 0)
       (effects (font (size 1.27 1.27)) (justify left))
     )
@@
       (effects (font (size 1.27 1.27)) (justify left))
     )
-    (property "Value" "1u" (id 1) (at 101.6 39.37 0)
+    (property "Value" "0.1f" (id 1) (at 101.6 39.37 0)
       (effects (font (size 1.27 1.27)) (justify left))
     )

Commit message: Finished PCB
Parts:
- C19, C20, C21, C22, C23, C24: footprint Capacitor_SMD:C_0805_2012Metric -> RamenKeebs:C_0805
Changed lines of the file:
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@@
   (title_block
     (title "Ramen80")
-    (date "2022-02-24")
+    (date "2022-03-05")
     (rev "v1.0.0")
     (company "Ramen Keebs")
@@
       (effects (font (size 1.27 1.27)) (justify left))
     )
-    (property "Footprint" "Capacitor_SMD:C_0805_2012Metric" (id 2) (at 74.6252 40.64 0)
+    (property "Footprint" "RamenKeebs:C_0805" (id 2) (at 74.6252 40.64 0)
       (effects (font (size 1.27 1.27)) hide)
     )
@@
       (effects (font (size 1.27 1.27)) (justify left))
     )
-    (property "Footprint" "Capacitor_SMD:C_0805_2012Metric" (id 2) (at 47.9552 40.64 0)
+    (property "Footprint" "RamenKeebs:C_0805" (id 2) (at 47.9552 40.64 0)
       (effects (font (size 1.27 1.27)) hide)
     )
@@
       (effects (font (size 1.27 1.27)) (justify left))
     )
-    (property "Footprint" "Capacitor_SMD:C_0805_2012Metric" (id 2) (at 56.8452 40.64 0)
+    (property "Footprint" "RamenKeebs:C_0805" (id 2) (at 56.8452 40.64 0)
       (effects (font (size 1.27 1.27)) hide)
     )
@@
       (effects (font (size 1.27 1.27)) (justify left))
     )
-    (property "Footprint" "Capacitor_SMD:C_0805_2012Metric" (id 2) (at 65.7352 40.64 0)
+    (property "Footprint" "RamenKeebs:C_0805" (id 2) (at 65.7352 40.64 0)
       (effects (font (size 1.27 1.27)) hide)
     )
@@
       (effects (font (size 1.27 1.27)) (justify left))
     )
-    (property "Footprint" "Capacitor_SMD:C_0805_2012Metric" (id 2) (at 83.5152 40.64 0)
+    (property "Footprint" "RamenKeebs:C_0805" (id 2) (at 83.5152 40.64 0)
       (effects (font (size 1.27 1.27)) hide)
     )
@@
       (effects (font (size 1.27 1.27)) (justify left))
     )
-    (property "Footprint" "Capacitor_SMD:C_0805_2012Metric" (id 2) (at 101.2952 40.64 0)
+    (property "Footprint" "RamenKeebs:C_0805" (id 2) (at 101.2952 40.64 0)
       (effects (font (size 1.27 1.27)) hide)
     )

Commit message: Created Gerber Files
Parts:
- C19, C21: value 0.47f -> 0.1µF
- C20: value 0.1f -> 0.1µF
- C22: value 0.1u -> 0.1µF
- C23: value 0.47f -> 4.7µF
- C24: value 0.1f -> 1µF
Changed lines of the file:
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@@
       (effects (font (size 1.27 1.27)) (justify left))
     )
-    (property "Value" "0.1u" (id 1) (at 74.93 39.37 0)
+    (property "Value" "0.1µF" (id 1) (at 74.93 39.37 0)
       (effects (font (size 1.27 1.27)) (justify left))
     )
@@
       (effects (font (size 1.27 1.27)) (justify left))
     )
-    (property "Value" "0.47f" (id 1) (at 48.26 39.37 0)
+    (property "Value" "0.1µF" (id 1) (at 48.26 39.37 0)
       (effects (font (size 1.27 1.27)) (justify left))
     )
@@
       (effects (font (size 1.27 1.27)) (justify left))
     )
-    (property "Value" "0.1f" (id 1) (at 57.15 39.37 0)
+    (property "Value" "0.1µF" (id 1) (at 57.15 39.37 0)
       (effects (font (size 1.27 1.27)) (justify left))
     )
@@
       (effects (font (size 1.27 1.27)) (justify left))
     )
-    (property "Value" "0.47f" (id 1) (at 66.04 39.37 0)
+    (property "Value" "0.1µF" (id 1) (at 66.04 39.37 0)
       (effects (font (size 1.27 1.27)) (justify left))
     )
@@
       (effects (font (size 1.27 1.27)) (justify left))
     )
-    (property "Value" "0.47f" (id 1) (at 83.82 39.37 0)
+    (property "Value" "4.7µF" (id 1) (at 83.82 39.37 0)
       (effects (font (size 1.27 1.27)) (justify left))
     )
@@
       (effects (font (size 1.27 1.27)) (justify left))
     )
-    (property "Value" "0.1f" (id 1) (at 101.6 39.37 0)
+    (property "Value" "1µF" (id 1) (at 101.6 39.37 0)
       (effects (font (size 1.27 1.27)) (justify left))
     )
