File: projects/Ramen80/Ramen80(Clock Crystal).kicad_sch (KiCad schematic)
At the start: 3 parts, among them Y1 FA-238_16.0000MB-C3

Commit message: Finished PCB
Parts:
- C25, C26: footprint Capacitor_SMD:C_0805_2012Metric -> RamenKeebs:C_0805
Changed lines of the file:
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@@
   (title_block
     (title "Ramen80")
-    (date "2022-02-24")
+    (date "2022-03-05")
     (rev "v1.0.0")
     (company "Ramen Keebs")
@@
       (effects (font (size 1.27 1.27)) (justify left))
     )
-    (property "Footprint" "Capacitor_SMD:C_0805_2012Metric" (id 2) (at 119.0752 85.09 0)
+    (property "Footprint" "RamenKeebs:C_0805" (id 2) (at 119.0752 85.09 0)
       (effects (font (size 1.27 1.27)) hide)
     )
@@
       (effects (font (size 1.27 1.27)) (justify left))
     )
-    (property "Footprint" "Capacitor_SMD:C_0805_2012Metric" (id 2) (at 169.8752 85.09 0)
+    (property "Footprint" "RamenKeebs:C_0805" (id 2) (at 169.8752 85.09 0)
       (effects (font (size 1.27 1.27)) hide)
     )

Commit message: Created Gerber Files
Parts:
- C25, C26: value C -> 22pF
Changed lines of the file:
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@@
       (effects (font (size 1.27 1.27)) (justify left))
     )
-    (property "Value" "C" (id 1) (at 119.38 83.82 0)
+    (property "Value" "22pF" (id 1) (at 119.38 83.82 0)
       (effects (font (size 1.27 1.27)) (justify left))
     )
@@
       (effects (font (size 1.27 1.27)) (justify left))
     )
-    (property "Value" "C" (id 1) (at 170.18 83.82 0)
+    (property "Value" "22pF" (id 1) (at 170.18 83.82 0)
       (effects (font (size 1.27 1.27)) (justify left))
     )
