File: projects/Ramen80/Ramen80(Led Matrix).kicad_sch (KiCad schematic)
At the start: 113 parts, among them U2 IS31FL3733-TQ, U3 IS31FL3733-TQ

Commit message: Reverted Pin Out Changes
Connections:
- net 2CS1: now also LED42.4 (VCC), LED72.4 (VCC), LED9.4 (VCC); no longer LED16.4 (VCC), LED49.4 (VCC)
- net 2CS10: now also LED26.4 (VCC), LED60.4 (VCC), LED82.4 (VCC); no longer LED30.4 (VCC), LED50.4 (VCC)
- net 2CS12: now also LED28.4 (VCC), LED62.4 (VCC), LED84.4 (VCC); no longer LED29.4 (VCC), LED63.4 (VCC), LED85.4 (VCC)
- net 2CS13: now also LED29.4 (VCC), LED63.4 (VCC), LED85.4 (VCC); no longer LED26.4 (VCC), LED60.4 (VCC), LED82.4 (VCC)
- net 2CS14: now also LED30.4 (VCC), LED50.4 (VCC); no longer LED31.4 (VCC), LED33.4 (VCC), LED86.4 (VCC)
- net 2CS15: now also LED31.4 (VCC), LED33.4 (VCC), LED86.4 (VCC); no longer LED25.4 (VCC), LED59.4 (VCC), LED81.4 (VCC)
- net 2CS2: now also LED10.4 (VCC), LED43.4 (VCC), LED73.4 (VCC); no longer LED11.4 (VCC), LED44.4 (VCC), LED74.4 (VCC)
- net 2CS3: now also LED11.4 (VCC), LED44.4 (VCC), LED74.4 (VCC); no longer LED15.4 (VCC), LED48.4 (VCC), LED76.4 (VCC)
- net 2CS4: now also LED12.4 (VCC), LED45.4 (VCC), LED75.4 (VCC); no longer LED14.4 (VCC), LED47.4 (VCC)
- net 2CS5: now also LED13.4 (VCC), LED46.4 (VCC); no longer LED10.4 (VCC), LED43.4 (VCC), LED73.4 (VCC)
- net 2CS6: now also LED14.4 (VCC), LED47.4 (VCC); no longer LED13.4 (VCC), LED46.4 (VCC)
- net 2CS7: now also LED15.4 (VCC), LED48.4 (VCC), LED76.4 (VCC); no longer LED12.4 (VCC), LED45.4 (VCC), LED75.4 (VCC)
- net 2CS8: now also LED16.4 (VCC), LED49.4 (VCC); no longer LED42.4 (VCC), LED72.4 (VCC), LED9.4 (VCC)
- net 2CS9 : now also LED25.4 (VCC), LED59.4 (VCC), LED81.4 (VCC); no longer LED28.4 (VCC), LED62.4 (VCC), LED84.4 (VCC)
- net CS1: now also LED1.4 (VCC), LED34.4 (VCC), LED64.4 (VCC); no longer LED41.4 (VCC), LED71.4 (VCC), LED8.4 (VCC)
- net CS2: now also LED2.4 (VCC), LED35.4 (VCC), LED65.4 (VCC); no longer LED40.4 (VCC), LED7.4 (VCC), LED70.4 (VCC)
- net CS3: now also LED3.4 (VCC), LED36.4 (VCC), LED66.4 (VCC); no longer LED39.4 (VCC), LED6.4 (VCC), LED69.4 (VCC)
- net CS4: now also LED37.4 (VCC), LED4.4 (VCC), LED67.4 (VCC); no longer LED38.4 (VCC), LED5.4 (VCC), LED68.4 (VCC)
- net CS5: now also LED38.4 (VCC), LED5.4 (VCC), LED68.4 (VCC); no longer LED37.4 (VCC), LED4.4 (VCC), LED67.4 (VCC)
- net CS6: now also LED39.4 (VCC), LED6.4 (VCC), LED69.4 (VCC); no longer LED3.4 (VCC), LED36.4 (VCC), LED66.4 (VCC)
- net CS7: now also LED40.4 (VCC), LED7.4 (VCC), LED70.4 (VCC); no longer LED2.4 (VCC), LED35.4 (VCC), LED65.4 (VCC)
- net CS8: now also LED41.4 (VCC), LED71.4 (VCC), LED8.4 (VCC); no longer LED1.4 (VCC), LED34.4 (VCC), LED64.4 (VCC)

Commit message: Finished PCB
Parts:
- C1, C10, C11, C12, C13, C14, C15, C16, C17, C18, C2, C3, C4, C5, C6, C7, C8, C9: footprint Capacitor_SMD:C_0805_2012Metric -> RamenKeebs:C_0805
- R1, R2, R3, R4, R5, R6: footprint Resistor_SMD:R_0805_2012Metric -> RamenKeebs:R_0805
Changed lines of the file:
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@@
   (title_block
     (title "Ramen80")
-    (date "2022-02-24")
+    (date "2022-03-05")
     (rev "v1.0.0")
     (company "Ramen Keebs")
@@
     (property "Reference" "C18" (id 0) (at 350.52 99.06 90))
     (property "Value" "0.1f" (id 1) (at 350.52 101.6 90))
-    (property "Footprint" "Capacitor_SMD:C_0805_2012Metric" (id 2) (at 354.33 105.7148 0)
+    (property "Footprint" "RamenKeebs:C_0805" (id 2) (at 354.33 105.7148 0)
       (effects (font (size 1.27 1.27)) hide)
     )
@@
       (effects (font (size 1.27 1.27)) (justify right))
     )
-    (property "Footprint" "Capacitor_SMD:C_0805_2012Metric" (id 2) (at 367.3348 66.04 0)
+    (property "Footprint" "RamenKeebs:C_0805" (id 2) (at 367.3348 66.04 0)
       (effects (font (size 1.27 1.27)) hide)
     )
@@
       (effects (font (size 1.27 1.27)) (justify right))
     )
-    (property "Footprint" "Capacitor_SMD:C_0805_2012Metric" (id 2) (at 390.1948 44.45 0)
+    (property "Footprint" "RamenKeebs:C_0805" (id 2) (at 390.1948 44.45 0)
       (effects (font (size 1.27 1.27)) hide)
     )
@@
       (effects (font (size 1.27 1.27)) (justify left))
     )
-    (property "Footprint" "Capacitor_SMD:C_0805_2012Metric" (id 2) (at 385.1148 66.04 0)
+    (property "Footprint" "RamenKeebs:C_0805" (id 2) (at 385.1148 66.04 0)
       (effects (font (size 1.27 1.27)) hide)
     )
@@
       (effects (font (size 1.27 1.27)) (justify right))
     )
-    (property "Footprint" "Capacitor_SMD:C_0805_2012Metric" (id 2) (at 367.3348 44.45 0)
+    (property "Footprint" "RamenKeebs:C_0805" (id 2) (at 367.3348 44.45 0)
       (effects (font (size 1.27 1.27)) hide)
     )
@@
       (effects (font (size 1.27 1.27)) (justify right))
     )
-    (property "Footprint" "Capacitor_SMD:C_0805_2012Metric" (id 2) (at 344.4748 66.04 0)
+    (property "Footprint" "RamenKeebs:C_0805" (id 2) (at 344.4748 66.04 0)
       (effects (font (size 1.27 1.27)) hide)
     )
@@
       (effects (font (size 1.27 1.27)) (justify left))
     )
-    (property "Footprint" "Capacitor_SMD:C_0805_2012Metric" (id 2) (at 362.2548 44.45 0)
+    (property "Footprint" "RamenKeebs:C_0805" (id 2) (at 362.2548 44.45 0)
       (effects (font (size 1.27 1.27)) hide)
     )
@@
       (effects (font (size 1.27 1.27)) (justify right))
     )
-    (property "Footprint" "Resistor_SMD:R_0805_2012Metric" (id 2) (at 59.182 207.01 90)
+    (property "Footprint" "RamenKeebs:R_0805" (id 2) (at 59.182 207.01 90)
       (effects (font (size 1.27 1.27)) hide)
     )
@@
       (effects (font (size 1.27 1.27)) (justify right))
     )
-    (property "Footprint" "Resistor_SMD:R_0805_2012Metric" (id 2) (at 342.392 134.62 90)
+    (property "Footprint" "RamenKeebs:R_0805" (id 2) (at 342.392 134.62 90)
       (effects (font (size 1.27 1.27)) hide)
     )
@@
     (property "Reference" "C17" (id 0) (at 350.52 87.63 90))
     (property "Value" "0.47f" (id 1) (at 350.52 90.17 90))
-    (property "Footprint" "Capacitor_SMD:C_0805_2012Metric" (id 2) (at 354.33 94.2848 0)
+    (property "Footprint" "RamenKeebs:C_0805" (id 2) (at 354.33 94.2848 0)
       (effects (font (size 1.27 1.27)) hide)
     )
@@
       (effects (font (size 1.27 1.27)) (justify left))
     )
-    (property "Footprint" "Capacitor_SMD:C_0805_2012Metric" (id 2) (at 385.1148 44.45 0)
+    (property "Footprint" "RamenKeebs:C_0805" (id 2) (at 385.1148 44.45 0)
       (effects (font (size 1.27 1.27)) hide)
     )
@@
       (effects (font (size 1.27 1.27)) (justify left))
     )
-    (property "Footprint" "Resistor_SMD:R_0805_2012Metric" (id 2) (at 344.932 132.08 90)
+    (property "Footprint" "RamenKeebs:R_0805" (id 2) (at 344.932 132.08 90)
       (effects (font (size 1.27 1.27)) hide)
     )
@@
       (effects (font (size 1.27 1.27)) (justify left))
     )
-    (property "Footprint" "Capacitor_SMD:C_0805_2012Metric" (id 2) (at 339.3948 44.45 0)
+    (property "Footprint" "RamenKeebs:C_0805" (id 2) (at 339.3948 44.45 0)
       (effects (font (size 1.27 1.27)) hide)
     )
@@
       (effects (font (size 1.27 1.27)) (justify left))
     )
-    (property "Footprint" "Capacitor_SMD:C_0805_2012Metric" (id 2) (at 339.3948 66.04 0)
+    (property "Footprint" "RamenKeebs:C_0805" (id 2) (at 339.3948 66.04 0)
       (effects (font (size 1.27 1.27)) hide)
     )
@@
     (property "Reference" "R5" (id 0) (at 52.07 189.23 90))
     (property "Value" "10k" (id 1) (at 52.07 191.77 90))
-    (property "Footprint" "Resistor_SMD:R_0805_2012Metric" (id 2) (at 52.07 197.358 90)
+    (property "Footprint" "RamenKeebs:R_0805" (id 2) (at 52.07 197.358 90)
       (effects (font (size 1.27 1.27)) hide)
     )
@@
       (effects (font (size 1.27 1.27)) (justify right))
     )
-    (property "Footprint" "Capacitor_SMD:C_0805_2012Metric" (id 2) (at 390.1948 66.04 0)
+    (property "Footprint" "RamenKeebs:C_0805" (id 2) (at 390.1948 66.04 0)
       (effects (font (size 1.27 1.27)) hide)
     )
@@
       (effects (font (size 1.27 1.27)) (justify right))
     )
-    (property "Footprint" "Capacitor_SMD:C_0805_2012Metric" (id 2) (at 344.4748 44.45 0)
+    (property "Footprint" "RamenKeebs:C_0805" (id 2) (at 344.4748 44.45 0)
       (effects (font (size 1.27 1.27)) hide)
     )
@@
       (effects (font (size 1.27 1.27)) (justify left))
     )
-    (property "Footprint" "Capacitor_SMD:C_0805_2012Metric" (id 2) (at 316.5348 66.04 0)
+    (property "Footprint" "RamenKeebs:C_0805" (id 2) (at 316.5348 66.04 0)
       (effects (font (size 1.27 1.27)) hide)
     )
@@
     (property "Reference" "R1" (id 0) (at 55.88 60.96 90))
     (property "Value" "5k1" (id 1) (at 55.88 63.5 90))
-    (property "Footprint" "Resistor_SMD:R_0805_2012Metric" (id 2) (at 55.88 69.088 90)
+    (property "Footprint" "RamenKeebs:R_0805" (id 2) (at 55.88 69.088 90)
       (effects (font (size 1.27 1.27)) hide)
     )
@@
       (effects (font (size 1.27 1.27)) (justify left))
     )
-    (property "Footprint" "Capacitor_SMD:C_0805_2012Metric" (id 2) (at 362.2548 66.04 0)
+    (property "Footprint" "RamenKeebs:C_0805" (id 2) (at 362.2548 66.04 0)
       (effects (font (size 1.27 1.27)) hide)
     )
@@
       (effects (font (size 1.27 1.27)) (justify right))
     )
-    (property "Footprint" "Capacitor_SMD:C_0805_2012Metric" (id 2) (at 321.6148 66.04 0)
+    (property "Footprint" "RamenKeebs:C_0805" (id 2) (at 321.6148 66.04 0)
       (effects (font (size 1.27 1.27)) hide)
     )
@@
       (effects (font (size 1.27 1.27)) (justify right))
     )
-    (property "Footprint" "Capacitor_SMD:C_0805_2012Metric" (id 2) (at 321.6148 44.45 0)
+    (property "Footprint" "RamenKeebs:C_0805" (id 2) (at 321.6148 44.45 0)
       (effects (font (size 1.27 1.27)) hide)
     )
@@
       (effects (font (size 1.27 1.27)) (justify left))
     )
-    (property "Footprint" "Capacitor_SMD:C_0805_2012Metric" (id 2) (at 316.5348 44.45 0)
+    (property "Footprint" "RamenKeebs:C_0805" (id 2) (at 316.5348 44.45 0)
       (effects (font (size 1.27 1.27)) hide)
     )
@@
       (effects (font (size 1.27 1.27)) (justify right))
     )
-    (property "Footprint" "Resistor_SMD:R_0805_2012Metric" (id 2) (at 59.182 78.74 90)
+    (property "Footprint" "RamenKeebs:R_0805" (id 2) (at 59.182 78.74 90)
       (effects (font (size 1.27 1.27)) hide)
     )

Commit message: Created Gerber Files
Parts:
- C1, C11, C17, C3: value 0.47f -> 0.47µF
- C10, C14, C8: value 0.47f -> 0.1µF
- C12, C2, C6: value 0.1f -> 0.1µF
- C13, C5, C9: value 0.1u -> 0.47µF
- C15, C18, C7: value 0.1f -> 0.47µF
- C16: value 1u -> 0.1µF
- C4: value 4.7u -> 0.1µF
- R1: value 5k1 -> 100kΩ
- R2: value 22 -> 20kΩ
- R3: value 5k1 -> 2kΩ
- R4: value 22 -> 2kΩ
- R5: value 10k -> 100kΩ
- R6: value 10k -> 10kΩ
