File: projects/Ramen80/Ramen80(Resistor Grid).kicad_sch (KiCad schematic)
At the start: 2 parts

Commit message: Fixes continue...
Parts:
- R11: value 10k -> 100k
- R12: value 10k -> 20k
Changed lines of the file:
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@@
     (in_bom yes) (on_board yes)
     (property "Reference" "R12" (id 0) (at 71.12 36.83 90))
-    (property "Value" "10k" (id 1) (at 71.12 39.37 90))
+    (property "Value" "20k" (id 1) (at 71.12 39.37 90))
     (property "Footprint" "Resistor_SMD:R_0805_2012Metric" (id 2) (at 71.12 41.148 90)
       (effects (font (size 1.27 1.27)) hide)
@@
     (in_bom yes) (on_board yes)
     (property "Reference" "R11" (id 0) (at 71.12 31.75 90))
-    (property "Value" "10k" (id 1) (at 71.12 34.29 90))
+    (property "Value" "100k" (id 1) (at 71.12 34.29 90))
     (property "Footprint" "Resistor_SMD:R_0805_2012Metric" (id 2) (at 71.12 36.068 90)
       (effects (font (size 1.27 1.27)) hide)

Commit message: Finished PCB
Parts:
- R11, R12: footprint Resistor_SMD:R_0805_2012Metric -> RamenKeebs:R_0805
Changed lines of the file:
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@@
   (title_block
     (title "Ramen80")
-    (date "2022-02-24")
+    (date "2022-03-05")
     (rev "v1.0.0")
     (company "Ramen Keebs")
@@
     (property "Reference" "R12" (id 0) (at 71.12 36.83 90))
     (property "Value" "20k" (id 1) (at 71.12 39.37 90))
-    (property "Footprint" "Resistor_SMD:R_0805_2012Metric" (id 2) (at 71.12 41.148 90)
+    (property "Footprint" "RamenKeebs:R_0805" (id 2) (at 71.12 41.148 90)
       (effects (font (size 1.27 1.27)) hide)
     )
@@
     (property "Reference" "R11" (id 0) (at 71.12 31.75 90))
     (property "Value" "100k" (id 1) (at 71.12 34.29 90))
-    (property "Footprint" "Resistor_SMD:R_0805_2012Metric" (id 2) (at 71.12 36.068 90)
+    (property "Footprint" "RamenKeebs:R_0805" (id 2) (at 71.12 36.068 90)
       (effects (font (size 1.27 1.27)) hide)
     )

Commit message: Created Gerber Files
Parts:
- R11: value 100k -> 10kΩ
- R12: value 20k -> 10kΩ
Changed lines of the file:
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@@
     (in_bom yes) (on_board yes)
     (property "Reference" "R12" (id 0) (at 71.12 36.83 90))
-    (property "Value" "20k" (id 1) (at 71.12 39.37 90))
+    (property "Value" "10kΩ" (id 1) (at 71.12 39.37 90))
     (property "Footprint" "RamenKeebs:R_0805" (id 2) (at 71.12 41.148 90)
       (effects (font (size 1.27 1.27)) hide)
@@
     (in_bom yes) (on_board yes)
     (property "Reference" "R11" (id 0) (at 71.12 31.75 90))
-    (property "Value" "100k" (id 1) (at 71.12 34.29 90))
+    (property "Value" "10kΩ" (id 1) (at 71.12 34.29 90))
     (property "Footprint" "RamenKeebs:R_0805" (id 2) (at 71.12 36.068 90)
       (effects (font (size 1.27 1.27)) hide)
