File: projects/Ramen80/Ramen80(Usb C Receptacle).kicad_sch (KiCad schematic)
At the start: 5 parts, among them J2 USB_C_RECEPTACLE

Commit message: Finished PCB
Parts:
- removed J2: USB_C_RECEPTACLE, SamacSys_Parts:GCT_USB4105-GF-A, symbol RamenKeebs:USB4105-GF-A
- added J2: USB4505-03-0-A, RamenKeebs:USB4505-03-0-A, symbol RamenKeebs:USB4505-03-0-A
- R10, R7, R8, R9: footprint Resistor_SMD:R_0805_2012Metric -> RamenKeebs:R_0805
Connections:
- net Cap+: now also J2.A6 (DP1), J2.B6 (DP2)
- net Cap-: now also J2.A7 (DN1), J2.B7 (DN2)
- net GND: now also J2.B1_A12 (GND_B), J2.S1 (SHELL_GND), J2.S2 (SHELL_GND), J2.S3 (SHELL_GND), J2.S4 (SHELL_GND)
- net VCC: now also J2.A4_B9 (VBUS_A), J2.B4_A9 (VBUS_B)
- net at R8.1: now also J2.B5 (CC2)
- net at R7.2: now also J2.A5 (CC1)
Other:
- moved on the sheet: R10, R9

Commit message: Created Gerber Files
Parts:
- added F1: 500mA, Fuse:Fuse_0805_2012Metric, symbol Device:Fuse
- R10: value 20k -> 22Ω
- R7, R8: value 2k -> 5k1Ω
- R9: value 100k -> 22Ω
Connections:
- net VCC: now also F1.2; no longer J2.A4_B9 (VBUS_A), J2.B4_A9 (VBUS_B)
- new net Fuse: F1.1, J2.A4_B9 (VBUS_A), J2.B4_A9 (VBUS_B)
Changed lines of the file:
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@@
+    (stroke (width 0) (type default) (color 0 0 0 0))
+  )
+  (wire (pts (xy 78.74 95.25) (xy 81.28 95.25))
+    (stroke (width 0) (type default) (color 0 0 0 0))
+  )
+  (wire (pts (xy 68.58 95.25) (xy 71.12 95.25))
     (stroke (width 0) (type default) (color 0 0 0 0))
   )
@@
   (wire (pts (xy 67.31 85.09) (xy 71.12 85.09))
     (stroke (width 0) (type default) (color 0 0 0 0))
+  )
+  (label "Fuse" (at 92.71 43.18 0)
+    (effects (font (size 1.27 1.27)) (justify left bottom))
   )
   (label "Cap-" (at 57.15 55.88 180)
@@
     (effects (font (size 1.27 1.27)) (justify left bottom))
   )
+  (label "Fuse" (at 57.15 43.18 180)
+    (effects (font (size 1.27 1.27)) (justify right bottom))
+  )
   (label "Cap+" (at 67.31 82.55 180)
+    (effects (font (size 1.27 1.27)) (justify right bottom))
+  )
+  (label "Fuse" (at 68.58 95.25 180)
     (effects (font (size 1.27 1.27)) (justify right bottom))
   )
@@
     (in_bom yes) (on_board yes) (fields_autoplaced)
     (property "Reference" "R10" (id 0) (at 74.93 88.9 90))
-    (property "Value" "20k" (id 1) (at 74.93 91.44 90))
+    (property "Value" "22Ω" (id 1) (at 74.93 91.44 90))
     (property "Footprint" "RamenKeebs:R_0805" (id 2) (at 74.93 86.868 90)
       (effects (font (size 1.27 1.27)) hide)
@@
     (pin "1")
     (pin "2")
-  )
-  (symbol (lib_id "power:VCC") (at 57.15 43.18 90) (unit 1)
-    (in_bom yes) (on_board yes) (fields_autoplaced)
-    (property "Reference" "#PWR0102" (id 0) (at 60.96 43.18 0)
-      (effects (font (size 1.27 1.27)) hide)
-    )
-    (property "Value" "VCC" (id 1) (at 53.34 43.1799 90)
-      (effects (font (size 1.27 1.27)) (justify left))
-    )
-    (property "Footprint" "" (id 2) (at 57.15 43.18 0)
-      (effects (font (size 1.27 1.27)) hide)
-    )
-    (property "Datasheet" "" (id 3) (at 57.15 43.18 0)
-      (effects (font (size 1.27 1.27)) hide)
-    )
-    (pin "1")
   )
   (symbol (lib_id "power:GND") (at 95.25 68.58 90) (unit 1)
@@
     (in_bom yes) (on_board yes) (fields_autoplaced)
     (property "Reference" "R7" (id 0) (at 48.26 54.61 90))
-    (property "Value" "2k" (id 1) (at 48.26 57.15 90))
+    (property "Value" "5k1Ω" (id 1) (at 48.26 57.15 90))
     (property "Footprint" "RamenKeebs:R_0805" (id 2) (at 48.26 52.578 90)
       (effects (font (size 1.27 1.27)) hide)
@@
     (pin "2")
   )
+  (symbol (lib_id "power:VCC") (at 81.28 95.25 270) (unit 1)
+    (in_bom yes) (on_board yes) (fields_autoplaced)
+    (property "Reference" "#PWR0102" (id 0) (at 77.47 95.25 0)
+      (effects (font (size 1.27 1.27)) hide)
+    )
+    (property "Value" "VCC" (id 1) (at 85.09 95.2499 90)
+      (effects (font (size 1.27 1.27)) (justify left))
+    )
+    (property "Footprint" "" (id 2) (at 81.28 95.25 0)
+      (effects (font (size 1.27 1.27)) hide)
+    )
+    (property "Datasheet" "" (id 3) (at 81.28 95.25 0)
+      (effects (font (size 1.27 1.27)) hide)
+    )
+    (pin "1")
+  )
   (symbol (lib_id "Device:R") (at 100.33 58.42 90) (unit 1)
     (in_bom yes) (on_board yes) (fields_autoplaced)
-    (property "Reference" "R8" (id 0) (at 100.33 52.07 90))
-    (property "Value" "2k" (id 1) (at 100.33 54.61 90))
+    (property "Reference" "R8" (id 0) (at 100.33 62.23 90))
+    (property "Value" "5k1Ω" (id 1) (at 100.33 64.77 90))
     (property "Footprint" "RamenKeebs:R_0805" (id 2) (at 100.33 60.198 90)
       (effects (font (size 1.27 1.27)) hide)
@@
     (in_bom yes) (on_board yes) (fields_autoplaced)
     (property "Reference" "R9" (id 0) (at 74.93 76.2 90))
-    (property "Value" "100k" (id 1) (at 74.93 78.74 90))
+    (property "Value" "22Ω" (id 1) (at 74.93 78.74 90))
     (property "Footprint" "RamenKeebs:R_0805" (id 2) (at 74.93 84.328 90)
       (effects (font (size 1.27 1.27)) hide)
@@
     (pin "2")
   )
-  (symbol (lib_id "power:VCC") (at 92.71 43.18 270) (unit 1)
-    (in_bom yes) (on_board yes) (fields_autoplaced)
-    (property "Reference" "#PWR0104" (id 0) (at 88.9 43.18 0)
-      (effects (font (size 1.27 1.27)) hide)
-    )
-    (property "Value" "VCC" (id 1) (at 96.52 43.1799 90)
-      (effects (font (size 1.27 1.27)) (justify left))
-    )
-    (property "Footprint" "" (id 2) (at 92.71 43.18 0)
-      (effects (font (size 1.27 1.27)) hide)
-    )
-    (property "Datasheet" "" (id 3) (at 92.71 43.18 0)
-      (effects (font (size 1.27 1.27)) hide)
-    )
-    (pin "1")
+  (symbol (lib_id "Device:Fuse") (at 74.93 95.25 90) (unit 1)
+    (in_bom yes) (on_board yes) (fields_autoplaced)
+    (property "Reference" "F1" (id 0) (at 74.93 99.06 90))
+    (property "Value" "500mA" (id 1) (at 74.93 101.6 90))
+    (property "Footprint" "Fuse:Fuse_0805_2012Metric" (id 2) (at 74.93 97.028 90)
+      (effects (font (size 1.27 1.27)) hide)
+    )
+    (property "Datasheet" "~" (id 3) (at 74.93 95.25 0)
+      (effects (font (size 1.27 1.27)) hide)
+    )
+    (pin "1")
+    (pin "2")
   )
 )
