File: projects/Ramen80/Ramen80.kicad_sch (KiCad schematic)
At the start: 1 part, among them U1 ATMEGA32U4

Commit message: Finished PCB
Parts:
- U1: footprint Keebio-Parts:ATMEGA32U4-AU -> RamenKeebs:ATMEGA32U4-AUR

Commit message: Created Gerber Files
Other:
- moved on the sheet: U1
